File: Shutdown_Circuit_Indicators.kicad_sch (KiCad schematic)
At the start: 5 parts

Commit message: Add files via upload
Updated Datasheet
Parts:
- R1: value 200 -> 400
Changed lines of the file:
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@@
     (in_bom yes) (on_board yes) (fields_autoplaced)
     (property "Reference" "R1" (id 0) (at 113.03 90.17 90))
-    (property "Value" "200" (id 1) (at 113.03 92.71 90))
+    (property "Value" "400" (id 1) (at 113.03 92.71 90))
     (property "Footprint" "Resistor_SMD:R_0603_1608Metric_Pad0.98x0.95mm_HandSolder" (id 2) (at 113.03 98.298 90)
       (effects (font (size 1.27 1.27)) hide)
     )
-    (property "Datasheet" "~" (id 3) (at 113.03 96.52 0)
+    (property "Datasheet" "https://www.mouser.com/datasheet/2/427/pat-1764170.pdf" (id 3) (at 113.03 96.52 0)
       (effects (font (size 1.27 1.27)) hide)
     )
@@
     )
     (path "/de6e164d-189b-467f-851b-5fff0c475288"
-      (reference "R1") (unit 1) (value "200") (footprint "Resistor_SMD:R_0603_1608Metric_Pad0.98x0.95mm_HandSolder")
+      (reference "R1") (unit 1) (value "400") (footprint "Resistor_SMD:R_0603_1608Metric_Pad0.98x0.95mm_HandSolder")
     )
     (path "/ee9190c7-2ff3-4b02-a619-4377fc17a2df"

Commit message: Add files via upload
Parts:
- R1: value 400 -> 1k
Changed lines of the file:
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@@
     (in_bom yes) (on_board yes) (fields_autoplaced)
     (property "Reference" "R1" (id 0) (at 113.03 90.17 90))
-    (property "Value" "400" (id 1) (at 113.03 92.71 90))
+    (property "Value" "1k" (id 1) (at 113.03 92.71 90))
     (property "Footprint" "Resistor_SMD:R_0603_1608Metric_Pad0.98x0.95mm_HandSolder" (id 2) (at 113.03 98.298 90)
       (effects (font (size 1.27 1.27)) hide)
     )
-    (property "Datasheet" "https://www.mouser.com/datasheet/2/427/pat-1764170.pdf" (id 3) (at 113.03 96.52 0)
+    (property "Datasheet" "https://datasheet.lcsc.com/lcsc/1811081617_YAGEO-RC0603JR-0710KL_C99198.pdf" (id 3) (at 113.03 96.52 0)
       (effects (font (size 1.27 1.27)) hide)
     )
@@
     )
     (path "/de6e164d-189b-467f-851b-5fff0c475288"
-      (reference "R1") (unit 1) (value "400") (footprint "Resistor_SMD:R_0603_1608Metric_Pad0.98x0.95mm_HandSolder")
+      (reference "R1") (unit 1) (value "1k") (footprint "Resistor_SMD:R_0603_1608Metric_Pad0.98x0.95mm_HandSolder")
     )
     (path "/ee9190c7-2ff3-4b02-a619-4377fc17a2df"

Commit message: Add files via upload
Parts:
- removed TP1: V_source-, TestPoint:TestPoint_Loop_D2.50mm_Drill1.0mm, symbol Connector:TestPoint
- removed TP2: V_source+, TestPoint:TestPoint_Loop_D2.50mm_Drill1.0mm, symbol Connector:TestPoint
- removed TP3: Ground, TestPoint:TestPoint_Loop_D2.50mm_Drill1.0mm, symbol Connector:TestPoint
- added J1, J2: 436500200, Global Libraries:436500200, symbol Global_Library:436500200
Connections:
- net Ground: now also J1.2
- net V_source+ renamed Input Power
- net Input Power: now also J1.1, J2.1
- no-connect marks 0 -> 1
Changed lines of the file:
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@@
   (junction (at 104.14 96.52) (diameter 0) (color 0 0 0 0)
   )
+  (no_connect (at 52.07 115.57))
   (wire (pts (xy 116.84 107.95) (xy 116.84 111.76))
-    (stroke (width 0) (type default) (color 0 0 0 0))
-  )
-  (wire (pts (xy 110.49 124.46) (xy 110.49 129.54))
-    (stroke (width 0) (type default) (color 0 0 0 0))
-  )
-  (wire (pts (xy 128.27 124.46) (xy 128.27 129.54))
-    (stroke (width 0) (type default) (color 0 0 0 0))
-  )
-  (wire (pts (xy 95.25 124.46) (xy 95.25 129.54))
     (stroke (width 0) (type default) (color 0 0 0 0))
   )
@@
     (stroke (width 0) (type default) (color 0 0 0 0))
   )
-  (global_label "Ground" (shape input) (at 128.27 129.54 270) (fields_autoplaced)
-    (effects (font (size 1.27 1.27)) (justify right))
-    (property "Intersheet References" "${INTERSHEET_REFS}" (id 0) (at 128.1906 138.6055 90)
-      (effects (font (size 1.27 1.27)) (justify right) hide)
-    )
-  )
   (global_label "Ground" (shape input) (at 116.84 111.76 0) (fields_autoplaced)
     (effects (font (size 1.27 1.27)) (justify left))
@@
     )
   )
-  (global_label "V_source-" (shape input) (at 99.06 111.76 180) (fields_autoplaced)
+  (global_label "Output Power" (shape input) (at 99.06 111.76 180) (fields_autoplaced)
     (effects (font (size 1.27 1.27)) (justify right))
-    (property "Intersheet References" "${INTERSHEET_REFS}" (id 0) (at 86.7288 111.8394 0)
+    (property "Intersheet References" "${INTERSHEET_REFS}" (id 0) (at 83.8259 111.6806 0)
       (effects (font (size 1.27 1.27)) (justify right) hide)
     )
   )
-  (global_label "V_source+" (shape input) (at 99.06 96.52 180) (fields_autoplaced)
+  (global_label "Input Power" (shape input) (at 99.06 96.52 180) (fields_autoplaced)
     (effects (font (size 1.27 1.27)) (justify right))
-    (property "Intersheet References" "${INTERSHEET_REFS}" (id 0) (at 86.7288 96.5994 0)
+    (property "Intersheet References" "${INTERSHEET_REFS}" (id 0) (at 85.2774 96.4406 0)
       (effects (font (size 1.27 1.27)) (justify right) hide)
     )
   )
-  (global_label "V_source-" (shape input) (at 95.25 129.54 270) (fields_autoplaced)
+  (global_label "Ground" (shape input) (at 52.07 105.41 180) (fields_autoplaced)
     (effects (font (size 1.27 1.27)) (justify right))
-    (property "Intersheet References" "${INTERSHEET_REFS}" (id 0) (at 95.3294 141.8712 90)
+    (property "Intersheet References" "${INTERSHEET_REFS}" (id 0) (at 43.0045 105.3306 0)
       (effects (font (size 1.27 1.27)) (justify right) hide)
     )
   )
-  (global_label "V_source+" (shape input) (at 110.49 129.54 270) (fields_autoplaced)
+  (global_label "Output Power" (shape input) (at 52.07 113.03 180) (fields_autoplaced)
     (effects (font (size 1.27 1.27)) (justify right))
-    (property "Intersheet References" "${INTERSHEET_REFS}" (id 0) (at 110.5694 141.8712 90)
+    (property "Intersheet References" "${INTERSHEET_REFS}" (id 0) (at 36.8359 112.9506 0)
       (effects (font (size 1.27 1.27)) (justify right) hide)
     )
   )
-  (symbol (lib_id "Connector:TestPoint") (at 110.49 124.46 0) (unit 1)
-    (in_bom yes) (on_board yes)
-    (property "Reference" "TP2" (id 0) (at 113.03 119.8879 0)
-      (effects (font (size 1.27 1.27)) (justify left))
+  (global_label "Input Power" (shape input) (at 52.07 102.87 180) (fields_autoplaced)
+    (effects (font (size 1.27 1.27)) (justify right))
+    (property "Intersheet References" "${INTERSHEET_REFS}" (id 0) (at 38.2874 102.7906 0)
+      (effects (font (size 1.27 1.27)) (justify right) hide)
     )
-    (property "Value" "V_source+" (id 1) (at 113.03 122.4279 0)
-      (effects (font (size 1.27 1.27)) (justify left))
+  )
+  (symbol (lib_id "Global_Library:436500200") (at 52.07 102.87 0) (unit 1)
+    (in_bom yes) (on_board yes) (fields_autoplaced)
+    (property "Reference" "J1" (id 0) (at 66.04 102.87 0)
+      (effects (font (size 1.524 1.524)) (justify left))
     )
-    (property "Footprint" "TestPoint:TestPoint_Loop_D2.50mm_Drill1.0mm" (id 2) (at 115.57 124.46 0)
-      (effects (font (size 1.27 1.27)) hide)
+    (property "Value" "436500200" (id 1) (at 66.04 106.68 0)
+      (effects (font (size 1.524 1.524)) (justify left))
     )
-    (property "Datasheet" "~" (id 3) (at 115.57 124.46 0)
-      (effects (font (size 1.27 1.27)) hide)
+    (property "Footprint" "Global Libraries:436500200" (id 2) (at 62.23 104.394 0)
+      (effects (font (size 1.524 1.524)) hide)
+    )
+    (property "Datasheet" "" (id 3) (at 52.07 102.87 0)
+      (effects (font (size 1.524 1.524)))
     )
     (pin "1")
+    (pin "2")
+  )
+  (symbol (lib_id "Global_Library:436500200") (at 52.07 113.03 0) (unit 1)
+    (in_bom yes) (on_board yes) (fields_autoplaced)
+    (property "Reference" "J2" (id 0) (at 66.04 113.03 0)
+      (effects (font (size 1.524 1.524)) (justify left))
+    )
+    (property "Value" "436500200" (id 1) (at 66.04 116.84 0)
+      (effects (font (size 1.524 1.524)) (justify left))
+    )
+    (property "Footprint" "Global Libraries:436500200" (id 2) (at 62.23 114.554 0)
+      (effects (font (size 1.524 1.524)) hide)
+    )
+    (property "Datasheet" "" (id 3) (at 52.07 113.03 0)
+      (effects (font (size 1.524 1.524)))
+    )
+    (pin "1")
+    (pin "2")
   )
   (symbol (lib_id "Device:LED") (at 116.84 104.14 90) (unit 1)
@@
     (pin "2")
   )
-  (symbol (lib_id "Connector:TestPoint") (at 128.27 124.46 0) (unit 1)
-    (in_bom yes) (on_board yes) (fields_autoplaced)
-    (property "Reference" "TP3" (id 0) (at 130.81 119.8879 0)
-      (effects (font (size 1.27 1.27)) (justify left))
-    )
-    (property "Value" "Ground" (id 1) (at 130.81 122.4279 0)
-      (effects (font (size 1.27 1.27)) (justify left))
-    )
-    (property "Footprint" "TestPoint:TestPoint_Loop_D2.50mm_Drill1.0mm" (id 2) (at 133.35 124.46 0)
-      (effects (font (size 1.27 1.27)) hide)
-    )
-    (property "Datasheet" "~" (id 3) (at 133.35 124.46 0)
-      (effects (font (size 1.27 1.27)) hide)
-    )
-    (pin "1")
-  )
   (symbol (lib_id "Device:R") (at 113.03 96.52 90) (unit 1)
     (in_bom yes) (on_board yes) (fields_autoplaced)
@@
     (pin "2")
   )
-  (symbol (lib_id "Connector:TestPoint") (at 95.25 124.46 0) (unit 1)
-    (in_bom yes) (on_board yes)
-    (property "Reference" "TP1" (id 0) (at 97.79 119.8879 0)
-      (effects (font (size 1.27 1.27)) (justify left))
-    )
-    (property "Value" "V_source-" (id 1) (at 97.79 122.4279 0)
-      (effects (font (size 1.27 1.27)) (justify left))
-    )
-    (property "Footprint" "TestPoint:TestPoint_Loop_D2.50mm_Drill1.0mm" (id 2) (at 100.33 124.46 0)
-      (effects (font (size 1.27 1.27)) hide)
-    )
-    (property "Datasheet" "~" (id 3) (at 100.33 124.46 0)
-      (effects (font (size 1.27 1.27)) hide)
-    )
-    (pin "1")
-  )
   (sheet_instances
     (path "/" (page "1"))
@@
       (reference "D1") (unit 1) (value "LED") (footprint "Diode_THT:D_T-1_P5.08mm_Horizontal")
     )
+    (path "/38ba0d6d-a7e2-436b-9565-8eb50c955d1b"
+      (reference "J1") (unit 1) (value "436500200") (footprint "Global Libraries:436500200")
+    )
+    (path "/8793c857-74d1-4c89-84fd-417db19c27e3"
+      (reference "J2") (unit 1) (value "436500200") (footprint "Global Libraries:436500200")
+    )
     (path "/de6e164d-189b-467f-851b-5fff0c475288"
       (reference "R1") (unit 1) (value "1k") (footprint "Resistor_SMD:R_0603_1608Metric_Pad0.98x0.95mm_HandSolder")
     )
-    (path "/ee9190c7-2ff3-4b02-a619-4377fc17a2df"
-      (reference "TP1") (unit 1) (value "V_source-") (footprint "TestPoint:TestPoint_Loop_D2.50mm_Drill1.0mm")
-    )
-    (path "/0451b222-e941-4943-8089-5824cc2844d5"
-      (reference "TP2") (unit 1) (value "V_source+") (footprint "TestPoint:TestPoint_Loop_D2.50mm_Drill1.0mm")
-    )
-    (path "/d9edf613-16a8-4142-9103-fbc6f8eb0dac"
-      (reference "TP3") (unit 1) (value "Ground") (footprint "TestPoint:TestPoint_Loop_D2.50mm_Drill1.0mm")
-    )
   )
